File: eagle/MHI-AC-Ctrl_v1.1.brd (EAGLE design)
At the start: 59.9 x 31.7 mm, 25 parts, among them U1 TSR_1-2450

Commit message: - refactored board
Parts:
- removed JP1: (no value), jumper:JP1
- removed TP1, TP14, TP15, TP16, TP2, TP3, TP4, TP5: TPPAD1-13, testpad:P1-13
- removed U$5: JST-PH_5-PIN_HEADER, srg:JST_B5B-PH_HEADER
- moved TP13 16.2 mm to (12.1, 13.0)
- moved C3 3.81 mm to (18.4, 26.0), turned to 180 degrees
- moved TP9 2.62 mm to (12.1, 5.08)
- moved U1 1.27 mm to (17.1, 19.1)
Connections:
- removed net N$10: TP2.TP, U$1.JP2.2
- removed net N$11: TP3.TP, U$1.JP2.3
- removed net N$12: TP4.TP, U$1.JP2.4
- removed net N$13: TP5.TP, U$1.JP2.5
- removed net N$86: JP1.1, U1.3
- removed net N$9: TP1.TP, U$1.JP2.1
- net +12V: no longer U$5.P1
- net +5V: now also U1.3; no longer JP1.2
- net GND: no longer TP14.TP, TP15.TP, TP16.TP, U$5.P5
- net MISO: no longer U$5.P4
- net MOSI: no longer U$5.P2
- net SCL: no longer U$5.P3
Routing:
- net +12V: track 38.2 -> 24.2 mm
- net N$86: track 8.25 -> 0.00 mm
- net GND: track 111.0 -> 106.7 mm
- net +5V: track 53.4 -> 49.8 mm
- net N$9: track 3.18 -> 0.00 mm
- net N$13: track 3.18 -> 0.00 mm
- net N$12: track 3.18 -> 0.00 mm
- net N$11: track 3.18 -> 0.00 mm
- net N$10: track 3.18 -> 0.00 mm
- net MOSI: track 46.1 -> 44.5 mm
- net MISO: track 44.6 -> 43.8 mm
Other:
- board text added: "September 2020"
- board text removed: "December 2019"
