File: eagle/MHI-AC-Ctrl_v1.1.sch (EAGLE design)
At the start: 25 parts, among them U1 TSR_1-2450

Commit message: - refactored board
Parts:
- removed JP1: (no value), jumper:JP1E
- removed TP1, TP14, TP15, TP16, TP2, TP3, TP4, TP5: TPPAD1-13, testpad:TPPAD1-13
- removed U$5: JST-PH_5-PIN_HEADER, srg:JST-PH_5-PIN_HEADER
Connections:
- removed net N$10: TP2.TP, U$1.RX
- removed net N$11: TP3.TP, U$1.D1
- removed net N$12: TP4.TP, U$1.D2
- removed net N$13: TP5.TP, U$1.D3
- removed net N$86: JP1.1, U1.VO
- removed net N$9: TP1.TP, U$1.TX
- net +12V: no longer U$5.1
- net +5V: now also U1.VO; no longer JP1.2
- net GND: no longer TP14.TP, TP15.TP, TP16.TP, U$5.5
- net MISO: no longer U$5.4
- net MOSI: no longer U$5.2
- net SCL: no longer U$5.3
Other:
- note removed: "only needed, for a second RC"
