File: eagle/MHI-AC-Ctrl_v1.2.brd (EAGLE design)
At the start: 59.9 x 31.7 mm, 15 parts, among them U1 TSR_1-2450

Commit message: - refactored board
Parts:
- removed TP6, TP7, TP8: TPPAD1-13, testpad:P1-13
- added R1: 4.7K, rcl:0204/7
- added U2: DS18B20, DS18B20:TO-92-TO92127P495H2044-3
- moved C1 1.27 mm to (5.71, 20.3)
- moved U1 1.27 mm to (17.1, 17.8)
- moved C3 0.64 mm to (18.4, 25.4)
Connections:
- net MISO_LV renamed N$1
- net MOSI_LV renamed N$2
- net +5V: now also R1.2, U2.3; no longer TP8.TP
- net GND: now also U2.1; no longer TP7.TP
- net N$14: now also R1.1, U2.2; no longer TP6.TP
Routing:
- net N$14: track 3.18 -> 37.4 mm
- net GND: track 106.7 -> 104.7 mm
- net +12V: track 24.2 -> 22.9 mm
- net +5V: track 49.8 -> 50.7 mm

Commit message: invert pin 2 and 3, remove AIRWIRE from DS18x20
Parts:
- moved TP11 3.25 mm to (14.6, 10.9)
- moved TP12 3.17 mm to (12.1, 8.89)
Connections:
- removed net MOSI: LS1.J2.6, TP12.TP, U$4.P2
- removed net SCL: LS1.J2.2, TP11.TP, U$4.P3
- new net N$3: LS1.J2.2, TP11.TP, U$4.P2
- new net N$4: LS1.J2.6, TP12.TP, U$4.P3
Routing:
- net N$4: track 0.00 -> 45.2 mm
- net MOSI: track 44.5 -> 0.00 mm
- net SCL: track 36.1 -> 0.00 mm
- net N$3: track 0.00 -> 34.2 mm
Changed lines of the file:
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@@
 <drawing>
 <settings>
-<setting alwaysvectorfont="yes"/>
+<setting alwaysvectorfont="no"/>
 <setting verticaltext="up"/>
 </settings>
@@
 <attribute name="VALUE" x="14.605" y="6.985" size="0.0254" layer="27"/>
 </element>
-<element name="TP11" library="testpad" library_urn="urn:adsk.eagle:library:385" package="P1-13" package3d_urn="urn:adsk.eagle:package:27946/1" value="TPPAD1-13" x="12.065" y="8.89" smashed="yes">
+<element name="TP11" library="testpad" library_urn="urn:adsk.eagle:library:385" package="P1-13" package3d_urn="urn:adsk.eagle:package:27946/1" value="TPPAD1-13" x="14.605" y="10.922" smashed="yes">
+<attribute name="NAME" x="13.589" y="12.192" size="1.27" layer="25" ratio="10"/>
+<attribute name="POPULARITY" value="12" x="14.605" y="10.922" size="1.778" layer="27" display="off"/>
+<attribute name="TP_SIGNAL_NAME" value="" x="14.605" y="10.922" size="1.778" layer="27" display="off"/>
+<attribute name="VALUE" x="14.605" y="10.922" size="0.0254" layer="27"/>
+</element>
+<element name="TP12" library="testpad" library_urn="urn:adsk.eagle:library:385" package="P1-13" package3d_urn="urn:adsk.eagle:package:27946/1" value="TPPAD1-13" x="12.065" y="8.89" smashed="yes">
 <attribute name="NAME" x="11.049" y="10.16" size="1.27" layer="25" ratio="10"/>
 <attribute name="POPULARITY" value="12" x="12.065" y="8.89" size="1.778" layer="27" display="off"/>
 <attribute name="TP_SIGNAL_NAME" value="" x="12.065" y="8.89" size="1.778" layer="27" display="off"/>
 <attribute name="VALUE" x="12.065" y="8.89" size="0.0254" layer="27"/>
-</element>
-<element name="TP12" library="testpad" library_urn="urn:adsk.eagle:library:385" package="P1-13" package3d_urn="urn:adsk.eagle:package:27946/1" value="TPPAD1-13" x="14.605" y="10.795" smashed="yes">
-<attribute name="NAME" x="13.589" y="12.065" size="1.27" layer="25" ratio="10"/>
-<attribute name="POPULARITY" value="12" x="14.605" y="10.795" size="1.778" layer="27" display="off"/>
-<attribute name="TP_SIGNAL_NAME" value="" x="14.605" y="10.795" size="1.778" layer="27" display="off"/>
-<attribute name="VALUE" x="14.605" y="10.795" size="0.0254" layer="27"/>
 </element>
 <element name="TP13" library="testpad" library_urn="urn:adsk.eagle:library:385" package="P1-13" package3d_urn="urn:adsk.eagle:package:27946/1" value="TPPAD1-13" x="12.065" y="12.954" smashed="yes">
@@
 <contactref element="U2" pad="1"/>
 <wire x1="17.145" y1="17.78" x2="17.0356" y2="17.6706" width="1.016" layer="16"/>
-<wire x1="17.145" y1="27.04998125" x2="17.0356" y2="27.15938125" width="0.8128" layer="16"/>
 <wire x1="17.145" y1="29.08475" x2="17.145" y2="25.4" width="0.8128" layer="16"/>
 <contactref element="LS1" pad="J1.4"/>
@@
 <wire x1="39.37" y1="9.525" x2="35.5725" y2="5.7275" width="1.143" layer="1"/>
 <wire x1="35.5725" y1="5.7275" x2="25.34969375" y2="5.7275" width="1.143" layer="1"/>
-<wire x1="17.145" y1="25.4" x2="17.145" y2="27.04998125" width="0" layer="19" extent="16-16"/>
 </signal>
 <signal name="+12V">
@@
 <wire x1="49.53" y1="22.225" x2="49.53" y2="23.495" width="1.016" layer="1"/>
 <contactref element="U1" pad="3"/>
-<wire x1="19.685" y1="25.4" x2="19.736" y2="25.451" width="1.016" layer="1"/>
 <wire x1="19.685" y1="25.4" x2="19.685" y2="21.59" width="1.016" layer="16"/>
 <wire x1="19.685" y1="21.59" x2="19.685" y2="17.78" width="1.016" layer="16"/>
@@
 <wire x1="36.83" y1="23.495" x2="36.83" y2="21.59" width="1.016" layer="16"/>
 </signal>
-<signal name="MOSI">
-<contactref element="LS1" pad="J2.6"/>
-<contactref element="TP12" pad="TP"/>
-<contactref element="U$4" pad="P2"/>
-<wire x1="14.51" y1="10.89" x2="14.605" y2="10.795" width="0.8128" layer="1"/>
-<wire x1="3.7625" y1="10.89" x2="14.51" y2="10.89" width="1.016" layer="16"/>
-<wire x1="14.51" y1="10.89" x2="14.605" y2="10.795" width="0.8128" layer="16"/>
-<wire x1="44.45" y1="19.685" x2="38.7604" y2="13.9954" width="1.016" layer="1"/>
-<wire x1="14.605" y1="10.795" x2="29.845" y2="10.795" width="1.016" layer="1"/>
-<wire x1="33.0454" y1="13.9954" x2="29.845" y2="10.795" width="1.016" layer="1"/>
-<wire x1="33.0454" y1="13.9954" x2="38.7604" y2="13.9954" width="1.016" layer="1"/>
-</signal>
 <signal name="MISO">
 <contactref element="U$4" pad="P4"/>
 <contactref element="LS1" pad="J2.5"/>
-<wire x1="26.035" y1="6.985" x2="35.56" y2="16.51" width="1.016" layer="16"/>
+<wire x1="35.56" y1="16.51" x2="26.035" y2="6.985" width="1.016" layer="16"/>
 <wire x1="35.56" y1="16.51" x2="36.83" y2="16.51" width="1.016" layer="16"/>
 <via x="36.83" y="16.51" extent="1-16" drill="0.6"/>
 <contactref element="TP10" pad="TP"/>
 <wire x1="14.51" y1="6.89" x2="14.605" y2="6.985" width="1.016" layer="1"/>
-<wire x1="3.7625" y1="6.89" x2="14.51" y2="6.89" width="1.016" layer="16"/>
-<wire x1="14.51" y1="6.89" x2="14.605" y2="6.985" width="1.016" layer="16"/>
-<wire x1="14.605" y1="6.985" x2="26.035" y2="6.985" width="1.016" layer="16"/>
 <wire x1="38.735" y1="16.3656" x2="36.9744" y2="16.3656" width="1.016" layer="1"/>
 <wire x1="36.83" y1="16.51" x2="36.9744" y2="16.3656" width="1.016" layer="1"/>
 <wire x1="41.91" y1="19.685" x2="38.735" y2="16.51" width="1.016" layer="1"/>
 <wire x1="38.735" y1="16.51" x2="38.735" y2="16.3656" width="1.016" layer="1"/>
+<wire x1="26.035" y1="6.985" x2="14.605" y2="6.985" width="1.016" layer="16"/>
+<wire x1="14.605" y1="6.985" x2="14.51" y2="6.89" width="1.016" layer="16"/>
+<wire x1="14.51" y1="6.89" x2="3.7625" y2="6.89" width="1.016" layer="16"/>
 </signal>
 <signal name="+3V3">
@@
 <wire x1="39.37" y1="5.08" x2="39.37" y2="3.175" width="0.8128" layer="16"/>
 <wire x1="35.56" y1="6.35" x2="38.1" y2="6.35" width="0.8128" layer="16"/>
-</signal>
-<signal name="SCL">
-<contactref element="U$4" pad="P3"/>
-<contactref element="LS1" pad="J2.2"/>
-<wire x1="34.29" y1="17.78" x2="25.4" y2="8.89" width="1.016" layer="16"/>
-<wire x1="34.29" y1="17.78" x2="34.29" y2="19.685" width="1.016" layer="16"/>
-<contactref element="TP11" pad="TP"/>
-<wire x1="3.7625" y1="8.89" x2="12.065" y2="8.89" width="1.016" layer="16"/>
-<wire x1="25.4" y1="8.89" x2="12.065" y2="8.89" width="1.016" layer="16"/>
 </signal>
 <signal name="N$14">
@@
 <wire x1="44.45" y1="9.525" x2="44.45" y2="3.175" width="1.016" layer="16"/>
 </signal>
+<signal name="N$3">
+<contactref element="LS1" pad="J2.2"/>
+<contactref element="TP11" pad="TP"/>
+<wire x1="34.29" y1="19.685" x2="25.527" y2="10.922" width="1.016" layer="16"/>
+<wire x1="25.527" y1="10.922" x2="14.605" y2="10.922" width="1.016" layer="16"/>
+<contactref element="U$4" pad="P2"/>
+<wire x1="3.7625" y1="10.89" x2="14.573" y2="10.89" width="1.016" layer="16"/>
+<wire x1="14.573" y1="10.89" x2="14.605" y2="10.922" width="1.016" layer="16"/>
+</signal>
+<signal name="N$4">
+<contactref element="U$4" pad="P3"/>
+<contactref element="LS1" pad="J2.6"/>
+<contactref element="TP12" pad="TP"/>
+<wire x1="12.065" y1="8.89" x2="3.7625" y2="8.89" width="1.016" layer="16"/>
+<wire x1="44.45" y1="19.685" x2="38.7604" y2="13.9954" width="1.016" layer="1"/>
+<wire x1="28.03805625" y1="8.89" x2="12.065" y2="8.89" width="1.016" layer="1"/>
+<wire x1="38.7604" y1="13.9954" x2="33.14345625" y2="13.9954" width="1.016" layer="1"/>
+<wire x1="33.14345625" y1="13.9954" x2="28.03805625" y2="8.89" width="1.016" layer="1"/>
+</signal>
 </signals>
