File: eagle/MHI-AC-Ctrl_v2.2.sch (EAGLE design)
At the start: 25 parts, among them U1 TSR_1-2450

Commit message: PCB layout update
Parts:
- removed JP1: (no value), jumper:JP1E
- removed TP1, TP10, TP11, TP12, TP13, TP14, TP15, TP16, TP2, TP3, TP4, TP5, TP6, TP7, TP8, TP9: TPPAD1-13, testpad:TPPAD1-13
- removed U$4, U$5: JST-PH_5-PIN_HEADER, srg:JST-PH_5-PIN_HEADER
- added R1: 4k7, rcl:R-EU_0207/10
- added X1: JST 03JQ-BT, Rembrandt Electronics - JST XH Connectors v1-0:JST-JQ-05-LONG-PAD
- added X3: JST-XH-03-PIN, Rembrandt Electronics - JST XH Connectors v1-0:JST-XH-03-PIN
- C1: value 22µ/50V -> 22µ/25V; device rcl:CPOL-EUE5-10.5 -> rcl:CPOL-EUE15-5AXIAL
- C3: value 22p -> 100n
Connections:
- removed net N$10: TP2.TP, U$1.RX
- removed net N$11: TP3.TP, U$1.D1
- removed net N$12: TP4.TP, U$1.D2
- removed net N$13: TP5.TP, U$1.D3
- removed net N$14: TP6.TP, U$1.D4
- removed net N$86: JP1.1, U1.VO
- removed net N$9: TP1.TP, U$1.TX
- removed net SCL: LS1.HV2, TP11.TP, U$4.3, U$5.3
- removed net SCL_LV: LS1.LV2, U$1.D5
- new net D2: R1.2, U$1.D2, X3-2.S
- new net SCK: LS1.HV3, X1-4.S
- new net SCK_LV: LS1.LV3, U$1.D5
- net +12V: now also C2.1, X1-5.S; no longer TP13.TP, U$4.1, U$5.1
- net +3V3: now also R1.1, X3-1.S
- net +5V: now also U1.VO; no longer C2.1, JP1.2, TP8.TP
- net GND: now also X1-1.S, X3-3.S; no longer TP14.TP, TP15.TP, TP16.TP, TP7.TP, TP9.TP, U$4.5, U$5.5
- net MISO: now also LS1.HV2, X1-2.S; no longer LS1.HV3, TP10.TP, U$4.4, U$5.4
- net MISO_LV: now also LS1.LV2; no longer LS1.LV3
- net MOSI: now also LS1.HV1, X1-3.S; no longer LS1.HV4, TP12.TP, U$4.2, U$5.2
- net MOSI_LV: now also LS1.LV1; no longer LS1.LV4
Other:
- note added: "MISO"
- note added: "MOSI"
- note added: "SCK"
- note added: "X1"
- note added: "to DS18x20"
- note removed: "only needed, for a second RC"
- moved on the sheet: C1, C2, C3, LS1
